File: HARDWARE/ESP32-DevKit-LiPo-Rev.B/ESP32-DevKit-Lipo_Rev_B.sch (KiCad schematic (older format))
At the start: 53 parts, among them Q1 Q12MHz/20pF/10ppm/4P/3.2x2.5mm, Q2 BC817-40(SOT23), Q3 BC817-40(SOT23), U1 BL4054B-42TPRN(SOT23-5), U2 CH340T(SSOP20W), U3 SY8089AAAC(SOT23-5), U5 ESP32-WROOM-32D-4MB

Commit message: Update
Parts:
- U1, U2, U5: Note (none) -> PB-Free
- U3: Fieldname 1 Value 1 -> (none); Fieldname2 Value2 -> (none); Fieldname3 Value3 -> (none); Note (none) -> PB-Free
